File: KiCadFile/speed radar.sch (KiCad schematic (older format))
At the start: 34 parts, among them J1 Conn_01x03, J2 Conn_01x03, J3 Conn_01x04, J4 Conn_01x03, U1 LM358, U2 ATmega328P-PU, U3 L78L05_TO92, Y1 16Mhz

Commit message: Add files via upload
Parts:
- R8: value 100M -> 100K
Changed lines of the file:
@@
 P 9050 2750
 F 0 "R8" V 9130 2750 50  0000 C CNN
-F 1 "100M" V 9050 2750 50  0000 C CNN
+F 1 "100K" V 9050 2750 50  0000 C CNN
 F 2 "Resistor_THT:R_Axial_DIN0207_L6.3mm_D2.5mm_P10.16mm_Horizontal" V 8980 2750 50  0001 C CNN
 F 3 "" H 9050 2750 50  0001 C CNN

Commit message: Add files via upload
Parts:
- R8: value 100K -> 200K
Changed lines of the file:
@@
 P 9050 2750
 F 0 "R8" V 9130 2750 50  0000 C CNN
-F 1 "100K" V 9050 2750 50  0000 C CNN
+F 1 "200K" V 9050 2750 50  0000 C CNN
 F 2 "Resistor_THT:R_Axial_DIN0207_L6.3mm_D2.5mm_P10.16mm_Horizontal" V 8980 2750 50  0001 C CNN
 F 3 "" H 9050 2750 50  0001 C CNN
